File: HW/WeatherStation_V2.kicad_pcb (KiCad board)
At the start: 2 copper layers, 74.9 x 61 mm, 61 parts, among them J1 Sensors + PWR, J2 I2C, J3 DHT, J4 I2C, J5 GPIO2, J6 I2C, J7 I2C, J8 BATTERY, J9 PROG, Q1 BC817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

Commit message: small improvements
Other:
- board text added: "Filada 06/2024"
- board text added: "I2C"
- board text added: "SCL"
- board text added: "SDA"
- board text removed: "Filada 11/2023"
Changed lines of the file:
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@@
     (property "ki_keywords" "connector")
     (attr through_hole)
-    (fp_text reference "J2" (at 3.75 -3.55 90) (layer "F.SilkS")
+    (fp_text reference "J2" (at 3.75 -3.55 90) (layer "F.SilkS") hide
         (effects (font (size 1 1) (thickness 0.15)))
     )
@@
     (property "ki_keywords" "connector")
     (attr through_hole)
-    (fp_text reference "J4" (at 3.75 -3.55 90) (layer "F.SilkS")
+    (fp_text reference "J4" (at 3.75 -3.55 90) (layer "F.SilkS") hide
         (effects (font (size 1 1) (thickness 0.15)))
     )
@@
     (property "ki_keywords" "connector")
     (attr through_hole)
-    (fp_text reference "J6" (at 3.75 -3.55 90) (layer "F.SilkS")
+    (fp_text reference "J6" (at 3.75 -3.55 90) (layer "F.SilkS") hide
         (effects (font (size 1 1) (thickness 0.15)))
     )
@@
     (property "ki_keywords" "connector")
     (attr through_hole)
-    (fp_text reference "J7" (at 3.75 -3.55 90) (layer "F.SilkS")
+    (fp_text reference "J7" (at 3.75 -3.55 90) (layer "F.SilkS") hide
         (effects (font (size 1 1) (thickness 0.15)))
     )
@@
     (effects (font (size 0.9 0.9) (thickness 0.14)) (justify left bottom))
   )
+  (gr_text "I2C" (at 189.6872 107.2388 90) (layer "F.SilkS")
+    (effects (font (size 1 1) (thickness 0.15)))
+  )
   (gr_text "DTR" (at 167.64 88.843964) (layer "F.SilkS")
     (effects (font (size 0.9 0.9) (thickness 0.14)) (justify left bottom))
   )
+  (gr_text "GND" (at 189.611 123.19 90) (layer "F.SilkS")
+    (effects (font (size 1 1) (thickness 0.15)))
+  )
   (gr_text "SDI" (at 151.13 111.703964 90) (layer "F.SilkS")
     (effects (font (size 0.9 0.9) (thickness 0.14)) (justify left bottom))
@@
     (effects (font (size 1 1) (thickness 0.15)) (justify left bottom))
   )
+  (gr_text "SDA" (at 189.611 129.54 90) (layer "F.SilkS")
+    (effects (font (size 1 1) (thickness 0.15)))
+  )
   (gr_text "WIND DIR" (at 126.365 100.908964 -90) (layer "F.SilkS")
     (effects (font (size 1 1) (thickness 0.125)) (justify left bottom))
   )
+  (gr_text "SCL" (at 189.611 132.715 90) (layer "F.SilkS")
+    (effects (font (size 1 1) (thickness 0.15)))
+  )
   (gr_text "WIND SPD" (at 126.365 81.223964 -90) (layer "F.SilkS")
     (effects (font (size 1 1) (thickness 0.125)) (justify left bottom))
@@
     (effects (font (size 0.9 0.9) (thickness 0.14)) (justify left bottom))
   )
+  (gr_text "3V3" (at 189.611 126.365 90) (layer "F.SilkS")
+    (effects (font (size 1 1) (thickness 0.15)))
+  )
   (gr_text "RAIN" (at 126.365 92.653964 -90) (layer "F.SilkS")
     (effects (font (size 1 1) (thickness 0.125)) (justify left bottom))
@@
     (effects (font (size 1.5 1.5) (thickness 0.3) bold) (justify left bottom))
   )
-  (gr_text "Filada 11/2023" (at 128.905 117.418964) (layer "F.Mask")
+  (gr_text "Filada 06/2024" (at 128.905 117.418964) (layer "F.Mask")
     (effects (font (size 1.5 1.5) (thickness 0.3) bold) (justify left bottom))
   )
